Commit message: Add launch file

File: urdf/wheelchair_simplified.urdf (robot description, URDF)
Before this commit: robot arlobot_hardware, 3 links, 2 joints
Joints:
- joint zed_footprint: child zed_center -> base_footprint; origin xyz=0.083 0 0.37 rpy=0 0 0 -> xyz=-0.385 0 -0.49 rpy=0 0 0; parent base_footprint -> zed_center

Commit message: Add csi_camera to wheelchair URDF

File: urdf/wheelchair_simplified.urdf (robot description, URDF)
Before this commit: robot arlobot_hardware, 3 links, 2 joints
Links:
- added link csi_cam, mass 0.01; collision cylinder length=0.005 radius=0.01; visual cylinder length=0.005 radius=0.01
Joints:
- added joint raspicam_footprint: type fixed, parent base_footprint, child raspicam, origin xyz=-0.24 0.05 0.926 rpy=1.5708 0 -1.5708

Commit message: Update URDF of wheelchair with Jetson

File: urdf/wheelchair_simplified.urdf (robot description, URDF)
Before this commit: robot arlobot_hardware, 4 links, 3 joints
Joints:
- removed joint raspicam_footprint
- added joint cam_footprint: type fixed, parent base_footprint, child csi_cam, origin xyz=-0.24 0.05 0.926 rpy=1.5708 0 -1.5708
- joint zed_footprint: origin xyz=-0.385 0 -0.49 rpy=0 0 0 -> xyz=-0.385 0 0 rpy=0 0 0
